File: kicad/CosmicWatch-ventidue.kicad_sch (KiCad schematic)
At the start: 19 parts, among them J101 Conn_01x05, J102 Conn_01x07, J103 Conn_01x05, J104 Conn_01x07, J105 Conn_01x05, J106 Conn_01x07, J107 Conn_01x05, J108 Conn_01x07, J109 BMP280, J110 Conn_01x06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

Commit message: Updated PCB files and added plots
Parts:
- BZ101: LCSC (none) -> C76871
- D101: footprint Package_TO_SOT_SMD:SOT-666 -> CosmicWatchPro:SOT-666; LCSC (none) -> C73592
- J110: value Conn_01x06 -> Mini GPS
- R102: LCSC (none) -> C17513
- R105, R106: LCSC (none) -> C17414
Connections:
- net VCC: now reaches U101.VIN
- no-connect marks 21 -> 20

Commit message: Push to version 3.3
Parts:
- U101: footprint CosmicWatchPro:Teensy4.1 -> CosmicWatchPro:Teensy4.1_Minimal; symbol CosmicWatchPro:Teensy4.1 -> CosmicWatchPro:Teensy4.1_minimal
Connections:
- net +3.3V: no longer U101.3.3V_3 (3.3V__2)
- net GND: no longer U101.GND4 (GND__3)
- removed net +5V: U101.5V
- no-connect marks 20 -> 13
Other:
- moved on the sheet: J109, J111, J112
