File: kicad/detector.kicad_sch (KiCad schematic)
At the start: 36 parts, among them J301 Conn_SMA, J302 Conn_SMA, J303 Conn_SMA, J304 Conn_SMA, U301 LT1807, U302 LT1807

Commit message: Updated PCB files and added plots
Parts:
- C301, C304, C305, C307: LCSC (none) -> C24666
- C302, C306: LCSC (none) -> C89258
- C303, C310: LCSC (none) -> C89190
- C308, C309: LCSC (none) -> C501858
- C311, C312: LCSC (none) -> C51574
- D301: LCSC (none) -> C905854
- D302: footprint Package_TO_SOT_SMD:SOT-666 -> CosmicWatchPro:SOT-666; LCSC (none) -> C73592
- J301, J302, J303, J304: LCSC (none) -> C88374
- R301, R302: LCSC (none) -> C2828807
- R303: LCSC (none) -> C96347
- R304, R307: LCSC (none) -> C17471
- R305: LCSC (none) -> C17522
- R306, R310: LCSC (none) -> C17414
- R308: LCSC (none) -> C17513
- R309, R311, R312, R313: LCSC (none) -> C149504
- U301, U302: LCSC (none) -> C665379
Changed lines of the file:
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@@
     (title "Detector PCB")
     (date "2022-07-14")
-    (rev "2.3")
+    (rev "2.5")
     (comment 1 "Pulse extenders are used to sample the event's intensity via the Teensy's analog I/O")
     (comment 2 "Two stages of amplification are used, with different amplification factors")
@@
       (effects (font (size 1.27 1.27)) hide)
     )
+    (property "LCSC" "C17414" (id 4) (at 198.12 105.41 0)
+      (effects (font (size 1.27 1.27)) hide)
+    )
     (pin "1")
     (pin "2")
@@
       (effects (font (size 1.27 1.27)) hide)
     )
+    (property "LCSC" "C24666" (id 4) (at 68.58 101.6 0)
+      (effects (font (size 1.27 1.27)) hide)
+    )
     (pin "1")
     (pin "2")
@@
       (effects (font (size 1.27 1.27)) hide)
     )
+    (property "LCSC" "C17414" (id 4) (at 154.94 102.87 0)
+      (effects (font (size 1.27 1.27)) hide)
+    )
     (pin "1")
     (pin "2")
@@
     )
     (property "Datasheet" "~" (id 3) (at 252.73 107.95 0)
+      (effects (font (size 1.27 1.27)) hide)
+    )
+    (property "LCSC" "C51574" (id 4) (at 252.73 107.95 0)
       (effects (font (size 1.27 1.27)) hide)
     )
@@
     (property "Datasheet" "" (id 3) (at 175.26 99.06 0)
       (effects (font (size 1.27 1.27)) (justify left bottom) hide)
+    )
+    (property "LCSC" "C665379" (id 4) (at 175.26 99.06 0)
+      (effects (font (size 1.27 1.27)) hide)
     )
     (pin "1")
@@
       (effects (font (size 1.27 1.27)) hide)
     )
+    (property "LCSC" "C149504" (id 4) (at 176.53 69.85 0)
+      (effects (font (size 1.27 1.27)) hide)
+    )
     (pin "1")
     (pin "2")
@@
     )
     (property "Datasheet" " ~" (id 3) (at 95.25 123.19 0)
+      (effects (font (size 1.27 1.27)) hide)
+    )
+    (property "LCSC" "C88374" (id 4) (at 95.25 123.19 0)
       (effects (font (size 1.27 1.27)) hide)
     )
@@
       (effects (font (size 1.27 1.27)) hide)
     )
+    (property "LCSC" "C89190" (id 4) (at 191.77 99.06 0)
+      (effects (font (size 1.27 1.27)) hide)
+    )
     (pin "1")
     (pin "2")
@@
       (effects (font (size 1.27 1.27)) hide)
     )
+    (property "LCSC" "C96347" (id 4) (at 120.65 50.8 0)
+      (effects (font (size 1.27 1.27)) hide)
+    )
     (pin "1")
     (pin "2")
@@
     )
     (property "Datasheet" "~" (id 3) (at 50.8 40.64 0)
+      (effects (font (size 1.27 1.27)) hide)
+    )
+    (property "LCSC" "C89190" (id 4) (at 50.8 40.64 0)
       (effects (font (size 1.27 1.27)) hide)
     )
@@
     (property "Datasheet" "" (id 3) (at 140.97 46.99 0)
       (effects (font (size 1.27 1.27)) (justify left bottom) hide)
+    )
+    (property "LCSC" "C665379" (id 4) (at 140.97 46.99 0)
+      (effects (font (size 1.27 1.27)) hide)
     )
     (pin "1")
@@
       (effects (font (size 1.27 1.27)) hide)
     )
+    (property "LCSC" "C2828807" (id 4) (at 44.45 34.29 0)
+      (effects (font (size 1.27 1.27)) hide)
+    )
     (pin "1")
     (pin "2")
@@
       (effects (font (size 1.27 1.27)) hide)
     )
+    (property "LCSC" "C149504" (id 4) (at 207.01 63.5 0)
+      (effects (font (size 1.27 1.27)) hide)
+    )
     (pin "1")
     (pin "2")
@@
       (effects (font (size 1.27 1.27)) hide)
     )
+    (property "LCSC" "C17522" (id 4) (at 138.43 55.88 0)
+      (effects (font (size 1.27 1.27)) hide)
+    )
     (pin "1")
     (pin "2")
@@
       (effects (font (size 1.27 1.27)) hide)
     )
+    (property "LCSC" "C89258" (id 4) (at 62.23 101.6 0)
+      (effects (font (size 1.27 1.27)) hide)
+    )
     (pin "1")
     (pin "2")
@@
     )
     (property "Datasheet" "~" (id 3) (at 125.73 62.23 0)
+      (effects (font (size 1.27 1.27)) hide)
+    )
+    (property "LCSC" "C17471" (id 4) (at 125.73 62.23 0)
       (effects (font (size 1.27 1.27)) hide)
     )
@@
       (effects (font (size 1.27 1.27)) hide)
     )
+    (property "LCSC" "C905854" (id 4) (at 91.44 39.37 0)
+      (effects (font (size 1.27 1.27)) hide)
+    )
     (pin "1")
     (pin "2")
@@
       (effects (font (size 1.27 1.27)) hide)
     )
+    (property "LCSC" "C88374" (id 4) (at 127 123.19 0)
+      (effects (font (size 1.27 1.27)) hide)
+    )
     (pin "1")
     (pin "2")
@@
       (effects (font (size 1.27 1.27)) hide)
     )
+    (property "LCSC" "C89258" (id 4) (at 39.37 101.6 0)
+      (effects (font (size 1.27 1.27)) hide)
+    )
     (pin "1")
     (pin "2")
@@
     )
     (property "Datasheet" "~" (id 3) (at 160.02 114.3 0)
+      (effects (font (size 1.27 1.27)) hide)
+    )
+    (property "LCSC" "C17471" (id 4) (at 160.02 114.3 0)
       (effects (font (size 1.27 1.27)) hide)
     )
@@
       (effects (font (size 1.27 1.27)) hide)
     )
+    (property "LCSC" "C501858" (id 4) (at 172.72 113.03 0)
+      (effects (font (size 1.27 1.27)) hide)
+    )
     (pin "1")
     (pin "2")
@@
       (effects (font (size 1.27 1.27)) hide)
     )
+    (property "LCSC" "C17513" (id 4) (at 172.72 107.95 0)
+      (effects (font (size 1.27 1.27)) hide)
+    )
     (pin "1")
     (pin "2")
@@
     )
     (property "Datasheet" "~" (id 3) (at 218.44 55.88 0)
+      (effects (font (size 1.27 1.27)) hide)
+    )
+    (property "LCSC" "C51574" (id 4) (at 218.44 55.88 0)
       (effects (font (size 1.27 1.27)) hide)
     )
@@
     (property "Datasheet" "" (id 3) (at 186.69 49.53 0)
       (effects (font (size 1.27 1.27)) (justify left bottom) hide)
+    )
+    (property "LCSC" "C665379" (id 4) (at 140.97 46.99 0)
+      (effects (font (size 1.27 1.27)) hide)
     )
     (pin "1")
@@
       (effects (font (size 1.27 1.27)) (justify left bottom) hide)
     )
+    (property "LCSC" "C665379" (id 4) (at 55.88 113.03 0)
+      (effects (font (size 1.27 1.27)) hide)
+    )
     (pin "1")
     (pin "2")
@@
       (effects (font (size 1.27 1.27)) hide)
     )
+    (property "LCSC" "C24666" (id 4) (at 69.85 40.64 0)
+      (effects (font (size 1.27 1.27)) hide)
+    )
     (pin "1")
     (pin "2")
@@
       (effects (font (size 1.27 1.27)) hide)
     )
+    (property "LCSC" "C501858" (id 4) (at 138.43 60.96 0)
+      (effects (font (size 1.27 1.27)) hide)
+    )
     (pin "1")
     (pin "2")
@@
     (property "Reference" "D302" (id 0) (at 237.8075 95.25 0))
     (property "Value" "BAS70XY" (id 1) (at 237.8075 97.79 0))
-    (property "Footprint" "Package_TO_SOT_SMD:SOT-666" (id 2) (at 236.22 101.6 0)
+    (property "Footprint" "CosmicWatchPro:SOT-666" (id 2) (at 236.22 101.6 0)
       (effects (font (size 1.27 1.27)) hide)
     )
     (property "Datasheet" "~" (id 3) (at 236.22 101.6 0)
+      (effects (font (size 1.27 1.27)) hide)
+    )
+    (property "LCSC" "C73592" (id 4) (at 201.93 49.53 0)
       (effects (font (size 1.27 1.27)) hide)
     )
@@
       (effects (font (size 1.27 1.27)) hide)
     )
+    (property "LCSC" "C149504" (id 4) (at 210.82 121.92 0)
+      (effects (font (size 1.27 1.27)) hide)
+    )
     (pin "1")
     (pin "2")
@@
       (effects (font (size 1.27 1.27)) hide)
     )
+    (property "LCSC" "C149504" (id 4) (at 241.3 115.57 0)
+      (effects (font (size 1.27 1.27)) hide)
+    )
     (pin "1")
     (pin "2")
@@
     )
     (property "Datasheet" "~" (id 3) (at 57.15 40.64 0)
+      (effects (font (size 1.27 1.27)) hide)
+    )
+    (property "LCSC" "C24666" (id 4) (at 57.15 40.64 0)
       (effects (font (size 1.27 1.27)) hide)
     )
@@
     (property "Datasheet" "" (id 3) (at 220.98 101.6 0)
       (effects (font (size 1.27 1.27)) (justify left bottom) hide)
+    )
+    (property "LCSC" "C665379" (id 4) (at 220.98 101.6 0)
+      (effects (font (size 1.27 1.27)) hide)
     )
     (pin "1")
@@
       (effects (font (size 1.27 1.27)) hide)
     )
+    (property "LCSC" "C88374" (id 4) (at 127 109.22 0)
+      (effects (font (size 1.27 1.27)) hide)
+    )
     (pin "1")
     (pin "2")
@@
     )
     (property "Datasheet" "~" (id 3) (at 33.02 101.6 0)
+      (effects (font (size 1.27 1.27)) hide)
+    )
+    (property "LCSC" "C24666" (id 4) (at 33.02 101.6 0)
       (effects (font (size 1.27 1.27)) hide)
     )
@@
       (effects (font (size 1.27 1.27)) hide)
     )
+    (property "LCSC" "C2828807" (id 4) (at 63.5 34.29 0)
+      (effects (font (size 1.27 1.27)) hide)
+    )
     (pin "1")
     (pin "2")
@@
     (property "Reference" "D302" (id 0) (at 203.5175 43.18 0))
     (property "Value" "BAS70XY" (id 1) (at 203.5175 45.72 0))
-    (property "Footprint" "Package_TO_SOT_SMD:SOT-666" (id 2) (at 201.93 49.53 0)
+    (property "Footprint" "CosmicWatchPro:SOT-666" (id 2) (at 201.93 49.53 0)
       (effects (font (size 1.27 1.27)) hide)
     )
     (property "Datasheet" "~" (id 3) (at 201.93 49.53 0)
+      (effects (font (size 1.27 1.27)) hide)
+    )
+    (property "LCSC" "C73592" (id 4) (at 201.93 49.53 0)
       (effects (font (size 1.27 1.27)) hide)
     )
@@
     (property "Datasheet" "" (id 3) (at 50.8 113.03 0)
       (effects (font (size 1.27 1.27)) (justify left bottom) hide)
+    )
+    (property "LCSC" "C665379" (id 4) (at 140.97 46.99 0)
+      (effects (font (size 1.27 1.27)) hide)
     )
     (pin "1")
@@
       (effects (font (size 1.27 1.27)) hide)
     )
+    (property "LCSC" "C88374" (id 4) (at 95.25 107.95 0)
+      (effects (font (size 1.27 1.27)) hide)
+    )

Commit message: Push to version 3.3
Parts:
- U301, U302: footprint Package_SO:MSOP-8_3x3mm_P0.65mm -> Package_SO:SO-8_3.9x4.9mm_P1.27mm
Changed lines of the file:
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@@
     (title "Detector PCB")
     (date "2022-07-14")
-    (rev "2.5")
+    (rev "3.3")
     (comment 1 "Pulse extenders are used to sample the event's intensity via the Teensy's analog I/O")
     (comment 2 "Two stages of amplification are used, with different amplification factors")
@@
     (property "Reference" "U302" (id 0) (at 175.26 90.17 0))
     (property "Value" "LT1807" (id 1) (at 175.26 92.71 0))
-    (property "Footprint" "Package_SO:MSOP-8_3x3mm_P0.65mm" (id 2) (at 176.53 91.44 0)
+    (property "Footprint" "Package_SO:SO-8_3.9x4.9mm_P1.27mm" (id 2) (at 176.53 91.44 0)
       (effects (font (size 1.27 1.27)) (justify left bottom) hide)
     )
@@
     (property "Reference" "U301" (id 0) (at 140.97 38.1 0))
     (property "Value" "LT1807" (id 1) (at 140.97 40.64 0))
-    (property "Footprint" "Package_SO:MSOP-8_3x3mm_P0.65mm" (id 2) (at 142.24 39.37 0)
+    (property "Footprint" "Package_SO:SO-8_3.9x4.9mm_P1.27mm" (id 2) (at 142.24 39.37 0)
       (effects (font (size 1.27 1.27)) (justify left bottom) hide)
     )
@@
     (pin "3")
     (pin "4")
+    (pin "MP")
   )
   (symbol (lib_id "CosmicWatchPro:Conn_SMA") (at 127 123.19 0) (unit 1)
@@
     (property "Reference" "U301" (id 0) (at 186.69 40.64 0))
     (property "Value" "LT1807" (id 1) (at 186.69 43.18 0))
-    (property "Footprint" "Package_SO:MSOP-8_3x3mm_P0.65mm" (id 2) (at 187.96 41.91 0)
+    (property "Footprint" "Package_SO:SO-8_3.9x4.9mm_P1.27mm" (id 2) (at 187.96 41.91 0)
       (effects (font (size 1.27 1.27)) (justify left bottom) hide)
     )
@@
       (effects (font (size 1.27 1.27)) (justify left))
     )
-    (property "Footprint" "Package_SO:MSOP-8_3x3mm_P0.65mm" (id 2) (at 57.15 105.41 0)
+    (property "Footprint" "Package_SO:SO-8_3.9x4.9mm_P1.27mm" (id 2) (at 57.15 105.41 0)
       (effects (font (size 1.27 1.27)) (justify left bottom) hide)
     )
@@
     (property "Reference" "U302" (id 0) (at 220.98 92.71 0))
     (property "Value" "LT1807" (id 1) (at 220.98 95.25 0))
-    (property "Footprint" "Package_SO:MSOP-8_3x3mm_P0.65mm" (id 2) (at 222.25 93.98 0)
+    (property "Footprint" "Package_SO:SO-8_3.9x4.9mm_P1.27mm" (id 2) (at 222.25 93.98 0)
       (effects (font (size 1.27 1.27)) (justify left bottom) hide)
     )
@@
       (effects (font (size 1.27 1.27)) (justify left))
     )
-    (property "Footprint" "Package_SO:MSOP-8_3x3mm_P0.65mm" (id 2) (at 52.07 105.41 0)
+    (property "Footprint" "Package_SO:SO-8_3.9x4.9mm_P1.27mm" (id 2) (at 52.07 105.41 0)
       (effects (font (size 1.27 1.27)) (justify left bottom) hide)
     )
