File: kicad/ethernet.kicad_sch (KiCad schematic)
At the start: 2 parts, among them U501 J1B12111CCD

Commit message: Updated PCB files and added plots
Parts:
- C501: LCSC (none) -> C89258
Changed lines of the file:
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@@
   (title_block
     (date "2022-07-14")
-    (rev "2.3")
+    (rev "2.5")
   )
   (junction (at 38.1 43.18) (diameter 0) (color 0 0 0 0)
@@
       (effects (font (size 1.27 1.27)) hide)
     )
+    (property "LCSC" "C89258" (id 4) (at 38.1 54.61 0)
+      (effects (font (size 1.27 1.27)) hide)
+    )
