File: kicad/power.kicad_sch (KiCad schematic)
At the start: 21 parts, among them U401 TCR2EF, U402 MAX5025

Commit message: Updated PCB files and added plots
Parts:
- added J401: Conn_01x02, Connector_JST:JST_PH_B2B-PH-K_1x02_P2.00mm_Vertical, symbol Connector_Generic:Conn_01x02
- BT401: footprint Connector_JST:JST_PH_B2B-PH-K_1x02_P2.00mm_Vertical -> Connector_Molex:Molex_PicoBlade_53047-0210_1x02_P1.25mm_Vertical; LCSC (none) -> C518987
- C401, C402, C403, C404: LCSC (none) -> C89190
- C405, C406: value 1uF -> 1uF, 50V; LCSC (none) -> C111768
- C407: value 10nF -> 10nF, 50V; LCSC (none) -> C83170
- D401: LCSC (none) -> C1884550
- L401: LCSC (none) -> C113070
- R401: LCSC (none) -> C17770
- R402: LCSC (none) -> C17462
- R403: LCSC (none) -> C17408
- U402: value MAX5025 -> MAX5026; LCSC (none) -> C87603
Connections:
- net GND: now also J401.2 (Pin_2)
- new net VCC: J401.1 (Pin_1)

Commit message: Push to version 3.3
Parts:
- added C408: 100nF, Capacitor_SMD:C_0805_2012Metric_Pad1.18x1.45mm_HandSolder, symbol Device:C
- added R404: 3.3k, Resistor_SMD:R_0805_2012Metric_Pad1.20x1.40mm_HandSolder, symbol Device:R
- C403: value 1uF -> 47uF
- R401: value 6.65k -> 6.8k
- R402: value 147k -> 150k
Connections:
- net GND: now also C404.2, C408.2
- net VCC: now also C401.1, C404.1, L401.1, TP406.1, U401.1 (VIN), U402.5 (VIN), C408.1, R404.2
- removed net +5V: C401.1, C403.1, C404.1, TP406.1, U401.1 (VIN)
- new net: C403.1, R404.1
Other:
- moved on the sheet: C403, C405, C406, C407, D401, L401, R401, R402, R403, U402
